File: BMS_Slave_KiCad/analog_in.kicad_sch (KiCad schematic)
At the start: 58 parts, among them U1 ${PART NUMBER}, U2 AD8628ARTZ-R2, U3 ADG728BRUZ

Commit message: noget af diagram tegningen er opdateret, vi fortsætter
Parts:
- C1, C10, C11, C12, C13, C14, C15, C16, C17, C18, C19, C2, C20, C21, C22, C3, C4, C5, C6, C7, C8, C9: value ${CAPACITANCE}/${RATED VOLTAGE} -> 10 nF; footprint CAPC1608X08N -> Capacitor_SMD:C_0603_1608Metric
- R10, R11, R20, R21, R22, R23, R24, R25, R26, R27, R28, R29, R30, R32, R33, R34: value ${RESISTANCE} -> 0; footprint RESC1608X05N -> Resistor_SMD:R_0603_1608Metric
- R12, R13, R14, R15, R16, R17, R18, R19, R31: value ${RESISTANCE} -> 1K; footprint RESC1608X05N -> Resistor_SMD:R_0603_1608Metric
- R2, R3, R4, R5, R6, R7, R8, R9: value ${RESISTANCE} -> 10K; footprint RESC1608X05N -> Resistor_SMD:R_0603_1608Metric
