File: BMS_Slave_KiCad/eeprom.kicad_sch (KiCad schematic)
At the start: 4 parts, among them U11 M24M02-DWMN3TP/K

Commit message: noget af diagram tegningen er opdateret, vi fortsætter
Parts:
- C103: value ${CAPACITANCE}/${RATED VOLTAGE} -> 10 nF; footprint CAPC1608X08N -> Capacitor_SMD:C_0603_1608Metric
Changed lines of the file:
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@@
 			)
 		)
-		(property "Value" "${CAPACITANCE}/${RATED VOLTAGE}"
+		(property "Value" "10 nF"
 			(at 131.826 151.9682 0)
 			(effects
@@
 			)
 		)
-		(property "Footprint" "CAPC1608X08N"
+		(property "Footprint" "Capacitor_SMD:C_0603_1608Metric"
 			(at 129.54 154.7622 0)
 			(effects
