File: BMS_Slave_KiCad/input_filter.kicad_sch (KiCad schematic)
At the start: 59 parts

Commit message: noget af diagram tegningen er opdateret, vi fortsætter
Parts:
- C49, C50, C51, C52, C53, C54, C55, C56, C57, C58, C59, C60, C61, C62, C63, C64, C65, C66, C67, C68, C69, C70, C71, C72, C73, C74, C75, C76, C77, C78, C79, C80: value ${CAPACITANCE}/${RATED VOLTAGE} -> 10 nF; footprint CAPC1608X08N -> Capacitor_SMD:C_0603_1608Metric
- R110, R111, R112, R113, R114, R115, R116, R117, R126, R127, R128: value ${RESISTANCE} -> 0; footprint RESC1608X05N -> Resistor_SMD:R_0603_1608Metric
- R118, R119, R120, R121, R122, R123, R124, R125, R129, R130, R131, R132, R133, R134, R135, R136: value ${RESISTANCE} -> 10K; footprint RESC1608X05N -> Resistor_SMD:R_0603_1608Metric
