File: BMS_Slave_KiCad/slave-14-mc33775.kicad_sch (KiCad schematic)
At the start: 1 part

Commit message: noget af diagram tegningen er opdateret, vi fortsætter
Parts:
- R1: value ${RESISTANCE} -> 0; footprint RESC1608X05N -> Resistor_SMD:R_0603_1608Metric
Changed lines of the file:
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@@
 			)
 		)
-		(property "Value" "${RESISTANCE}"
+		(property "Value" "0"
 			(at 177.546 115.3922 0)
 			(effects
@@
 			)
 		)
-		(property "Footprint" "RESC1608X05N"
+		(property "Footprint" "Resistor_SMD:R_0603_1608Metric"
 			(at 175.26 111.5822 0)
 			(effects
