File: BMS_Slave_KiCad/connectors.kicad_sch (KiCad schematic)
At the start: 13 parts, among them J10 ${PART NUMBER}, J11 ${PART NUMBER}, J12 ${PART NUMBER}, J13 ${PART NUMBER}, J2 ${PART NUMBER}, J3 WR-MPC4 64901621122, J4 WR-MPC4 64901621122, J5 WR-MPC4 64900221122, J6 WR-MPC4 64900221122, J7 WR-MPC4 64900221122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

Commit message: Updated footprints - halfway done
Parts:
- J10, J9: value ${PART NUMBER} -> Pinheader_2x7_vertical; footprint Pinheader_2.54_2x7 -> Connector_PinHeader_2.54mm:PinHeader_2x07_P2.54mm_Vertical
- J11, J12, J2: value ${PART NUMBER} -> Pinheader_2x1_vertical; footprint Pinheader_2.54_2 -> Connector_PinHeader_2.54mm:PinHeader_1x02_P2.54mm_Vertical
- J13: value ${PART NUMBER} -> Pinheader_2x9_vertical; footprint Pinheader_2.54_2x9 -> Connector_PinHeader_2.54mm:PinHeader_2x09_P2.54mm_Vertical
Changed lines of the file:
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@@
 			)
 		)
-		(property "Value" "${PART NUMBER}"
+		(property "Value" "Pinheader_2x1_vertical"
 			(at 205.74 241.1222 0)
 			(effects
@@
 			)
 		)
-		(property "Footprint" "Pinheader_2.54_2"
+		(property "Footprint" "Connector_PinHeader_2.54mm:PinHeader_1x02_P2.54mm_Vertical"
 			(at 200.66 233.5022 0)
 			(effects
@@
 			)
 		)
-		(property "Value" "${PART NUMBER}"
+		(property "Value" "Pinheader_2x1_vertical"
 			(at 205.74 253.8222 0)
 			(effects
@@
 			)
 		)
-		(property "Footprint" "Pinheader_2.54_2"
+		(property "Footprint" "Connector_PinHeader_2.54mm:PinHeader_1x02_P2.54mm_Vertical"
 			(at 200.66 246.2022 0)
 			(effects
@@
 			)
 		)
-		(property "Value" "${PART NUMBER}"
+		(property "Value" "Pinheader_2x7_vertical"
 			(at 205.74 200.4822 0)
 			(effects
@@
 			)
 		)
-		(property "Footprint" "Pinheader_2.54_2x7"
+		(property "Footprint" "Connector_PinHeader_2.54mm:PinHeader_2x07_P2.54mm_Vertical"
 			(at 200.66 180.1622 0)
 			(effects
@@
 			)
 		)
-		(property "Value" "${PART NUMBER}"
+		(property "Value" "Pinheader_2x7_vertical"
 			(at 205.74 228.4222 0)
 			(effects
@@
 			)
 		)
-		(property "Footprint" "Pinheader_2.54_2x7"
+		(property "Footprint" "Connector_PinHeader_2.54mm:PinHeader_2x07_P2.54mm_Vertical"
 			(at 200.66 208.1022 0)
 			(effects
@@
 			)
 		)
-		(property "Value" "${PART NUMBER}"
+		(property "Value" "Pinheader_2x9_vertical"
 			(at 307.34 111.5822 0)
 			(effects
@@
 			)
 		)
-		(property "Footprint" "Pinheader_2.54_2x9"
+		(property "Footprint" "Connector_PinHeader_2.54mm:PinHeader_2x09_P2.54mm_Vertical"
 			(at 302.26 86.1822 0)
 			(effects
@@
 			)
 		)
-		(property "Value" "${PART NUMBER}"
+		(property "Value" "Pinheader_2x1_vertical"
 			(at 91.44 236.0422 0)
 			(effects
@@
 			)
 		)
-		(property "Footprint" "Pinheader_2.54_2"
+		(property "Footprint" "Connector_PinHeader_2.54mm:PinHeader_1x02_P2.54mm_Vertical"
 			(at 104.14 228.4222 0)
 			(effects
