File: BMS_Slave_KiCad/dcdc-converter.kicad_sch (KiCad schematic)
At the start: 29 parts, among them U12 ${PART NUMBER}

Commit message: noget af diagram tegningen er opdateret, vi fortsætter
Parts:
- 3.3V_DCDC1, Vin_DCDC1, enable_DCDC1: footprint Testpoint_S1 -> TestPoint:TestPoint_Pad_2.5x2.5mm
- C104, C105: value ${CAPACITANCE}/${RATED VOLTAGE} -> 15uF; footprint CAPC6153X67N -> KCM55WR72A156MH01K:CAPC6153X670N
- C106, C109, C111: value ${CAPACITANCE}/${RATED VOLTAGE} -> 2.2uF; footprint CAPC3225X25N -> Capacitor_SMD:C_1210_3225Metric
- C107: value ${CAPACITANCE}/${RATED VOLTAGE} -> 3.3uF; footprint CAPC4532X16N -> Capacitor_SMD:C_1812_4532Metric
- C108: value ${CAPACITANCE}/${RATED VOLTAGE} -> 10 nF; footprint CAPC1608X08N -> Capacitor_SMD:C_0603_1608Metric
- C110, C112, C113: value ${CAPACITANCE}/${RATED VOLTAGE} -> 22pF; footprint CAPC1005X06N -> Capacitor_SMD:C_0402_1005Metric
- C114: value ${CAPACITANCE}/${RATED VOLTAGE} -> 22u; footprint CAPC3216X18N -> Capacitor_SMD:C_1206_3216Metric
- R189, R191, R195: value ${RESISTANCE} -> 0; footprint RESC1608X05N -> Resistor_SMD:R_0603_1608Metric
- R190: value ${RESISTANCE} -> 10K; footprint RESC1608X05N -> Resistor_SMD:R_0603_1608Metric
Changed lines of the file:
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@@
 			)
 		)
-		(property "Value" "${CAPACITANCE}/${RATED VOLTAGE}"
+		(property "Value" "22pF"
 			(at 167.386 124.0282 0)
 			(effects
@@
 			)
 		)
-		(property "Footprint" "CAPC1005X06N"
+		(property "Footprint" "Capacitor_SMD:C_0402_1005Metric"
 			(at 165.1 119.2022 0)
 			(effects
@@
 			)
 		)
-		(property "Value" "${CAPACITANCE}/${RATED VOLTAGE}"
+		(property "Value" "2.2uF"
 			(at 164.846 68.1482 0)
 			(effects
@@
 			)
 		)
-		(property "Footprint" "CAPC3225X25N"
+		(property "Footprint" "Capacitor_SMD:C_1210_3225Metric"
 			(at 162.56 70.9422 0)
 			(effects
@@
 			)
 		)
-		(property "Value" "${CAPACITANCE}/${RATED VOLTAGE}"
+		(property "Value" "10 nF"
 			(at 93.726 126.5682 0)
 			(effects
@@
 			)
 		)
-		(property "Footprint" "CAPC1608X08N"
+		(property "Footprint" "Capacitor_SMD:C_0603_1608Metric"
 			(at 91.44 129.3622 0)
 			(effects
@@
 			)
 		)
-		(property "Footprint" "Testpoint_S1"
+		(property "Footprint" "TestPoint:TestPoint_Pad_2.5x2.5mm"
 			(at 281.94 124.2822 0)
 			(effects
@@
 			)
 		)
-		(property "Value" "${CAPACITANCE}/${RATED VOLTAGE}"
+		(property "Value" "22pF"
 			(at 195.326 136.7282 0)
 			(effects
@@
 			)
 		)
-		(property "Footprint" "CAPC1005X06N"
+		(property "Footprint" "Capacitor_SMD:C_0402_1005Metric"
 			(at 193.04 139.5222 0)
 			(effects
@@
 			)
 		)
-		(property "Value" "${RESISTANCE}"
+		(property "Value" "0"
 			(at 68.326 67.1322 0)
 			(effects
@@
 			)
 		)
-		(property "Footprint" "RESC1608X05N"
+		(property "Footprint" "Resistor_SMD:R_0603_1608Metric"
 			(at 66.04 63.3222 0)
 			(effects
@@
 			)
 		)
-		(property "Value" "${RESISTANCE}"
+		(property "Value" "10K"
 			(at 39.37 157.0482 0)
 			(effects
@@
 			)
 		)
-		(property "Footprint" "RESC1608X05N"
+		(property "Footprint" "Resistor_SMD:R_0603_1608Metric"
 			(at 38.1 149.6822 0)
 			(effects
@@
 			)
 		)
-		(property "Value" "${CAPACITANCE}/${RATED VOLTAGE}"
+		(property "Value" "22u"
 			(at 268.986 141.8082 0)
 			(effects
@@
 			)
 		)
-		(property "Footprint" "CAPC3216X18N"
+		(property "Footprint" "Capacitor_SMD:C_1206_3216Metric"
 			(at 266.7 144.6022 0)
 			(effects
@@
 			)
 		)
-		(property "Value" "${CAPACITANCE}/${RATED VOLTAGE}"
+		(property "Value" "15uF"
 			(at 58.166 68.1482 0)
 			(effects
@@
 			)
 		)
-		(property "Footprint" "CAPC6153X67N"
+		(property "Footprint" "KCM55WR72A156MH01K:CAPC6153X670N"
 			(at 55.88 70.9422 0)
 			(effects
@@
 			)
 		)
-		(property "Footprint" "Testpoint_S1"
+		(property "Footprint" "TestPoint:TestPoint_Pad_2.5x2.5mm"
 			(at 109.22 129.3622 0)
 			(effects
@@
 			)
 		)
-		(property "Value" "${RESISTANCE}"
+		(property "Value" "0"
 			(at 242.57 60.5282 0)
 			(effects
@@
 			)
 		)
-		(property "Footprint" "RESC1608X05N"
+		(property "Footprint" "Resistor_SMD:R_0603_1608Metric"
 			(at 241.3 63.3222 0)
 			(effects
@@
 			)
 		)
-		(property "Value" "${CAPACITANCE}/${RATED VOLTAGE}"
+		(property "Value" "2.2uF"
 			(at 177.546 68.1482 0)
 			(effects
@@
 			)
 		)
-		(property "Footprint" "CAPC3225X25N"
+		(property "Footprint" "Capacitor_SMD:C_1210_3225Metric"
 			(at 175.26 70.9422 0)
 			(effects
@@
 			)
 		)
-		(property "Value" "${RESISTANCE}"
+		(property "Value" "0"
 			(at 39.37 139.2682 0)
 			(effects
@@
 			)
 		)
-		(property "Footprint" "RESC1608X05N"
+		(property "Footprint" "Resistor_SMD:R_0603_1608Metric"
 			(at 38.1 131.9022 0)
 			(effects
@@
 			)
 		)
-		(property "Value" "${CAPACITANCE}/${RATED VOLTAGE}"
+		(property "Value" "3.3uF"
 			(at 86.106 73.2282 0)
 			(effects
@@
 			)
 		)
-		(property "Footprint" "CAPC4532X16N"
+		(property "Footprint" "Capacitor_SMD:C_1812_4532Metric"
 			(at 83.82 76.0222 0)
 			(effects
@@
 			)
 		)
-		(property "Value" "${CAPACITANCE}/${RATED VOLTAGE}"
+		(property "Value" "15uF"
 			(at 42.926 68.1482 0)
 			(effects
@@
 			)
 		)
-		(property "Footprint" "CAPC6153X67N"
+		(property "Footprint" "KCM55WR72A156MH01K:CAPC6153X670N"
 			(at 40.64 70.9422 0)
 			(effects
@@
 			)
 		)
-		(property "Value" "${CAPACITANCE}/${RATED VOLTAGE}"
+		(property "Value" "2.2uF"
 			(at 75.946 126.5682 0)
 			(effects
@@
 			)
 		)
-		(property "Footprint" "CAPC3225X25N"
+		(property "Footprint" "Capacitor_SMD:C_1210_3225Metric"
 			(at 73.66 129.3622 0)
 			(effects
@@
 			)
 		)
-		(property "Value" "${CAPACITANCE}/${RATED VOLTAGE}"
+		(property "Value" "22pF"
 			(at 205.486 134.1882 0)
 			(effects
@@
 			)
 		)
-		(property "Footprint" "CAPC1005X06N"
+		(property "Footprint" "Capacitor_SMD:C_0402_1005Metric"
 			(at 203.2 129.3622 0)
 			(effects
@@
 			)
 		)
-		(property "Footprint" "Testpoint_S1"
+		(property "Footprint" "TestPoint:TestPoint_Pad_2.5x2.5mm"
 			(at 104.14 119.2022 0)
 			(effects

Commit message: Updated footprints - halfway done
Parts:
- L1: value ${INDUCTANCE} -> 470nH; footprint SRP7028A -> Inductor_SMD:L_Bourns_SRP7028A_7.3x6.6mm
- L2: value ${INDUCTANCE} -> 47uH
- LD4: value ${COLOR} -> GREEN
Changed lines of the file:
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@@
 			)
 		)
-		(property "Value" "${COLOR}"
+		(property "Value" "GREEN"
 			(at 243.332 70.6882 0)
 			(effects
@@
 			)
 		)
-		(property "Value" "${INDUCTANCE}"
+		(property "Value" "47uH"
 			(at 193.04 127.8382 0)
 			(effects
@@
 			)
 		)
-		(property "Value" "${INDUCTANCE}"
+		(property "Value" "470nH"
 			(at 68.58 59.2582 0)
 			(effects
@@
 			)
 		)
-		(property "Footprint" "SRP7028A"
+		(property "Footprint" "Inductor_SMD:L_Bourns_SRP7028A_7.3x6.6mm"
 			(at 66.04 55.7022 0)
 			(effects
