File: BMS_Slave_KiCad/ldo.kicad_sch (KiCad schematic)
At the start: 12 parts, among them U10 ${PART NUMBER}, U9 ${PART NUMBER}

Commit message: noget af diagram tegningen er opdateret, vi fortsætter
Parts:
- 3.3V_LDO1: footprint Testpoint_S1 -> TestPoint:TestPoint_Pad_2.5x2.5mm
- C100, C101: value ${CAPACITANCE}/${RATED VOLTAGE} -> 10 nF; footprint CAPC1608X08N -> Capacitor_SMD:C_0603_1608Metric
- C102: value ${CAPACITANCE}/${RATED VOLTAGE} -> 2.2uF; footprint CAPC2012X14N -> Capacitor_SMD:C_0805_2012Metric
- R181, R183, R185: value ${RESISTANCE} -> 0; footprint RESC1608X05N -> Resistor_SMD:R_0603_1608Metric
Changed lines of the file:
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@@
 			)
 		)
-		(property "Footprint" "Testpoint_S1"
+		(property "Footprint" "TestPoint:TestPoint_Pad_2.5x2.5mm"
 			(at 254 121.7422 0)
 			(effects
@@
 			)
 		)
-		(property "Value" "${CAPACITANCE}/${RATED VOLTAGE}"
+		(property "Value" "10 nF"
 			(at 91.186 129.1082 0)
 			(effects
@@
 			)
 		)
-		(property "Footprint" "CAPC1608X08N"
+		(property "Footprint" "Capacitor_SMD:C_0603_1608Metric"
 			(at 88.9 131.9022 0)
 			(effects
@@
 			)
 		)
-		(property "Value" "${RESISTANCE}"
+		(property "Value" "0"
 			(at 107.95 131.6482 0)
 			(effects
@@
 			)
 		)
-		(property "Footprint" "RESC1608X05N"
+		(property "Footprint" "Resistor_SMD:R_0603_1608Metric"
 			(at 106.68 134.4422 0)
 			(effects
@@
 			)
 		)
-		(property "Value" "${RESISTANCE}"
+		(property "Value" "0"
 			(at 223.266 125.5522 0)
 			(effects
@@
 			)
 		)
-		(property "Footprint" "RESC1608X05N"
+		(property "Footprint" "Resistor_SMD:R_0603_1608Metric"
 			(at 220.98 121.7422 0)
 			(effects
@@
 			)
 		)
-		(property "Value" "${CAPACITANCE}/${RATED VOLTAGE}"
+		(property "Value" "10 nF"
 			(at 116.586 159.5882 0)
 			(effects
@@
 			)
 		)
-		(property "Footprint" "CAPC1608X08N"
+		(property "Footprint" "Capacitor_SMD:C_0603_1608Metric"
 			(at 114.3 162.3822 0)
 			(effects
@@
 			)
 		)
-		(property "Value" "${CAPACITANCE}/${RATED VOLTAGE}"
+		(property "Value" "2.2uF"
 			(at 190.246 131.6482 0)
 			(effects
@@
 			)
 		)
-		(property "Footprint" "CAPC2012X14N"
+		(property "Footprint" "Capacitor_SMD:C_0805_2012Metric"
 			(at 187.96 134.4422 0)
 			(effects
@@
 			)
 		)
-		(property "Value" "${RESISTANCE}"
+		(property "Value" "0"
 			(at 219.71 164.6682 0)
 			(effects
@@
 			)
 		)
-		(property "Footprint" "RESC1608X05N"
+		(property "Footprint" "Resistor_SMD:R_0603_1608Metric"
 			(at 218.44 167.4622 0)
 			(effects

Commit message: Updated footprints - halfway done
Parts:
- LD3: value ${COLOR} -> GREEN
Changed lines of the file:
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@@
 			)
 		)
-		(property "Value" "${COLOR}"
+		(property "Value" "GREEN"
 			(at 220.472 174.8282 0)
 			(effects
