File: BMS_Slave_KiCad/mc33775.kicad_sch (KiCad schematic)
At the start: 95 parts, among them Q1 ${PART NUMBER}, Q2 ${PART NUMBER}, Q3 ${PART NUMBER}, T1 ${PART NUMBER}, T2 ${PART NUMBER}, U7 ${PART NAME}, U8 ${PART NAME}

Commit message: noget af diagram tegningen er opdateret, vi fortsætter
Parts:
- ALARM_IN1, ALARM_OUT1, GND1, TPL_H_N1, TPL_H_P1, TPL_L_N1, TPL_L_P1, Vaux1, Vbat1, Vbat_con_ext1, Vddc1, Vmodule1: footprint Testpoint_S1 -> TestPoint:TestPoint_Pad_2.5x2.5mm
- C81, C83, C84, C85, C86, C87, C89, C90, C91, C92, C93, C94, C95, C97, C98: value ${CAPACITANCE}/${RATED VOLTAGE} -> 10 nF; footprint CAPC1608X08N -> Capacitor_SMD:C_0603_1608Metric
- C82, C88, C96, C99: value ${CAPACITANCE}/${RATED VOLTAGE} -> 22pF; footprint CAPC1005X06N -> Capacitor_SMD:C_0402_1005Metric
- D1, D11: value ${PART NUMBER} -> ~; footprint ON-SEMI-SOT-23-3-CASE-318-08 -> (none)
- R139, R140, R141, R142, R143, R144, R145, R146, R147, R148, R149, R150, R151, R152, R153, R154, R155, R156, R157, R158, R162, R170, R174, R176, R177, R178, R179, R180: value ${RESISTANCE} -> 0; footprint RESC1608X05N -> Resistor_SMD:R_0603_1608Metric

Commit message: Updated footprints - halfway done
Parts:
- D10, D2, D3: value ${PART NUMBER} -> Schottky_100V_1A; footprint PowerDI123 -> Diode_SMD:D_PowerDI-123
- D4: value ${PART NUMBER} -> PTVS60VS1UR; footprint NEXPERIA_PTVSxS1UR -> Diode_SMD:Nexperia_CFP3_SOD-123W
- D5: value ${PART NUMBER} -> S1MSP1-7; footprint S1MSP1 -> Diode_SMD:D_PowerDI-123
- D6, D7, D8, D9: value ${PART NUMBER} -> PESD5V0V1BB; footprint SOD523_PESD_NEXPERIA -> Diode_SMD:D_SOD-523
- LD1, LD2: value ${COLOR} -> GREEN
Changed lines of the file:
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@@
 			)
 		)
-		(property "Value" "${PART NUMBER}"
+		(property "Value" "Schottky_100V_1A"
 			(at 322.072 184.9882 0)
 			(effects
@@
 			)
 		)
-		(property "Footprint" "PowerDI123"
+		(property "Footprint" "Diode_SMD:D_PowerDI-123"
 			(at 320.04 187.7822 0)
 			(effects
@@
 			)
 		)
-		(property "Value" "${PART NUMBER}"
+		(property "Value" "PTVS60VS1UR"
 			(at 89.662 53.4162 0)
 			(effects
@@
 			)
 		)
-		(property "Footprint" "NEXPERIA_PTVSxS1UR"
+		(property "Footprint" "Diode_SMD:Nexperia_CFP3_SOD-123W"
 			(at 87.63 46.8122 0)
 			(effects
@@
 			)
 		)
-		(property "Value" "${PART NUMBER}"
+		(property "Value" "Schottky_100V_1A"
 			(at 32.766 37.4142 0)
 			(effects
@@
 			)
 		)
-		(property "Footprint" "PowerDI123"
+		(property "Footprint" "Diode_SMD:D_PowerDI-123"
 			(at 40.64 32.8422 0)
 			(effects
@@
 			)
 		)
-		(property "Value" "${PART NUMBER}"
+		(property "Value" "PESD5V0V1BB"
 			(at 272.796 141.5542 0)
 			(effects
@@
 			)
 		)
-		(property "Footprint" "SOD523_PESD_NEXPERIA"
+		(property "Footprint" "Diode_SMD:D_SOD-523"
 			(at 278.13 136.9822 0)
 			(effects
@@
 			)
 		)
-		(property "Value" "${PART NUMBER}"
+		(property "Value" "PESD5V0V1BB"
 			(at 272.796 172.0342 0)
 			(effects
@@
 			)
 		)
-		(property "Footprint" "SOD523_PESD_NEXPERIA"
+		(property "Footprint" "Diode_SMD:D_SOD-523"
 			(at 278.13 167.4622 0)
 			(effects
@@
 			)
 		)
-		(property "Value" "${COLOR}"
+		(property "Value" "GREEN"
 			(at 309.372 75.7682 0)
 			(effects
@@
 			)
 		)
-		(property "Value" "${PART NUMBER}"
+		(property "Value" "PESD5V0V1BB"
 			(at 272.796 161.8742 0)
 			(effects
@@
 			)
 		)
-		(property "Footprint" "SOD523_PESD_NEXPERIA"
+		(property "Footprint" "Diode_SMD:D_SOD-523"
 			(at 278.13 157.3022 0)
 			(effects
@@
 			)
 		)
-		(property "Value" "${COLOR}"
+		(property "Value" "GREEN"
 			(at 337.312 75.7682 0)
 			(effects
@@
 			)
 		)
-		(property "Value" "${PART NUMBER}"
+		(property "Value" "S1MSP1-7"
 			(at 111.252 54.1782 0)
 			(effects
@@
 			)
 		)
-		(property "Footprint" "S1MSP1"
+		(property "Footprint" "Diode_SMD:D_PowerDI-123"
 			(at 109.22 46.8122 0)
 			(effects
@@
 			)
 		)
-		(property "Value" "${PART NUMBER}"
+		(property "Value" "PESD5V0V1BB"
 			(at 272.796 131.3942 0)
 			(effects
@@
 			)
 		)
-		(property "Footprint" "SOD523_PESD_NEXPERIA"
+		(property "Footprint" "Diode_SMD:D_SOD-523"
 			(at 278.13 126.8222 0)
 			(effects
@@
 			)
 		)
-		(property "Value" "${PART NUMBER}"
+		(property "Value" "Schottky_100V_1A"
 			(at 32.766 47.5742 0)
 			(effects
@@
 			)
 		)
-		(property "Footprint" "PowerDI123"
+		(property "Footprint" "Diode_SMD:D_PowerDI-123"
 			(at 40.64 43.0022 0)
 			(effects
