File: BMS_Slave_KiCad/sensors.kicad_sch (KiCad schematic)
At the start: 11 parts, among them IC1 MCP9800A0T-M/OT, U13 ${PART NAME}, U14 ${PART NAME}, U15 BME280

Commit message: noget af diagram tegningen er opdateret, vi fortsætter
Parts:
- C115, C116, C117, C118, C119, C120: value ${CAPACITANCE}/${RATED VOLTAGE} -> 10 nF; footprint CAPC1608X08N -> Capacitor_SMD:C_0603_1608Metric
- R199: value ${RESISTANCE} -> 10K; footprint RESC1608X05N -> Resistor_SMD:R_0603_1608Metric
Changed lines of the file:
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@@
 			)
 		)
-		(property "Value" "${CAPACITANCE}/${RATED VOLTAGE}"
+		(property "Value" "10 nF"
 			(at 248.666 101.1682 0)
 			(effects
@@
 			)
 		)
-		(property "Footprint" "CAPC1608X08N"
+		(property "Footprint" "Capacitor_SMD:C_0603_1608Metric"
 			(at 246.38 103.9622 0)
 			(effects
@@
 			)
 		)
-		(property "Value" "${CAPACITANCE}/${RATED VOLTAGE}"
+		(property "Value" "10 nF"
 			(at 230.886 101.1682 0)
 			(effects
@@
 			)
 		)
-		(property "Footprint" "CAPC1608X08N"
+		(property "Footprint" "Capacitor_SMD:C_0603_1608Metric"
 			(at 228.6 103.9622 0)
 			(effects
@@
 			)
 		)
-		(property "Value" "${CAPACITANCE}/${RATED VOLTAGE}"
+		(property "Value" "10 nF"
 			(at 319.786 159.5882 0)
 			(effects
@@
 			)
 		)
-		(property "Footprint" "CAPC1608X08N"
+		(property "Footprint" "Capacitor_SMD:C_0603_1608Metric"
 			(at 317.5 162.3822 0)
 			(effects
@@
 			)
 		)
-		(property "Value" "${CAPACITANCE}/${RATED VOLTAGE}"
+		(property "Value" "10 nF"
 			(at 164.846 159.5882 0)
 			(effects
@@
 			)
 		)
-		(property "Footprint" "CAPC1608X08N"
+		(property "Footprint" "Capacitor_SMD:C_0603_1608Metric"
 			(at 162.56 162.3822 0)
 			(effects
@@
 			)
 		)
-		(property "Value" "${RESISTANCE}"
+		(property "Value" "10K"
 			(at 146.05 235.7882 0)
 			(effects
@@
 			)
 		)
-		(property "Footprint" "RESC1608X05N"
+		(property "Footprint" "Resistor_SMD:R_0603_1608Metric"
 			(at 144.78 238.5822 0)
 			(effects
@@
 			)
 		)
-		(property "Value" "${CAPACITANCE}/${RATED VOLTAGE}"
+		(property "Value" "10 nF"
 			(at 304.546 164.6682 0)
 			(effects
@@
 			)
 		)
-		(property "Footprint" "CAPC1608X08N"
+		(property "Footprint" "Capacitor_SMD:C_0603_1608Metric"
 			(at 302.26 167.4622 0)
 			(effects
@@
 			)
 		)
-		(property "Value" "${CAPACITANCE}/${RATED VOLTAGE}"
+		(property "Value" "10 nF"
 			(at 121.666 263.7282 0)
 			(effects
@@
 			)
 		)
-		(property "Footprint" "CAPC1608X08N"
+		(property "Footprint" "Capacitor_SMD:C_0603_1608Metric"
 			(at 129.54 258.9022 0)
 			(effects

Commit message: Updated footprints - halfway done
Parts:
- IC1: footprint SOT-23-OT5_L -> Package_TO_SOT_SMD:SOT-23-5
Changed lines of the file:
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@@
 			)
 		)
-		(property "Footprint" "SOT-23-OT5_L"
+		(property "Footprint" "Package_TO_SOT_SMD:SOT-23-5"
 			(at 114.3 238.5822 0)
 			(effects
