File: BMS_Slave_KiCad/slave-14-mc33775.kicad_pcb (KiCad board)
At the start: 6 copper layers, 160 x 1.3 mm, 38 parts

Commit message: Updated footprints - halfway done
Parts:
- removed R706, R707, R708, R709, R710, R711, R712, R713: ThermaWick, Vishay_THJP_0603:Vishay_THJP_0603
- removed R714, R715, R716, R717, R718, R719, R720, R721, R722, R723, R724, R725, R726, R727, R728, R729, R730, R731, R732, R733, R734, R735, R736, R737, R738, R739, R740, R741: 68R, RESC5025X07N:RESC5025X07N
- added 3.3V_DCDC1: Testpoint_Square, TestPoint:TestPoint_Pad_2.5x2.5mm, F.Cu at (139.5, 96.9)
- added 3.3V_LDO1: Testpoint_Square, TestPoint:TestPoint_Pad_2.5x2.5mm, F.Cu at (110.2, 145.5)
- added ALARM_IN1: Testpoint_Square, TestPoint:TestPoint_Pad_2.5x2.5mm, F.Cu at (78.1, 111.4)
- added ALARM_OUT1: Testpoint_Square, TestPoint:TestPoint_Pad_2.5x2.5mm, F.Cu at (78.1, 115.9)
- added C1: 10 nF, Capacitor_SMD:C_0603_1608Metric, F.Cu at (105.9, 87.8)
- added C10: 10 nF, Capacitor_SMD:C_0603_1608Metric, F.Cu at (105.9, 110.3)
- added C100: 10 nF, Capacitor_SMD:C_0603_1608Metric, F.Cu at (105.9, 144.5)
- added C101: 10 nF, Capacitor_SMD:C_0603_1608Metric, F.Cu at (105.9, 147.0)
- added C102: 2.2uF, Capacitor_SMD:C_0805_2012Metric, F.Cu at (110.2, 149.3)
- added C103: 10 nF, Capacitor_SMD:C_0603_1608Metric, F.Cu at (122.5, 144.5)
- added C106: 2.2uF, Capacitor_SMD:C_1210_3225Metric, F.Cu at (134.4, 96.8)
- added C107: 3.3uF, Capacitor_SMD:C_1812_4532Metric, F.Cu at (139.4, 89.0)
- added C108: 10 nF, Capacitor_SMD:C_0603_1608Metric, F.Cu at (143.8, 95.9)
- added C109: 2.2uF, Capacitor_SMD:C_1210_3225Metric, F.Cu at (134.4, 101.0)
- added C11: 10 nF, Capacitor_SMD:C_0603_1608Metric, F.Cu at (105.9, 112.8)
- added C110: 22pF, Capacitor_SMD:C_0402_1005Metric, F.Cu at (127.4, 99.0)
- added C111: 2.2uF, Capacitor_SMD:C_1210_3225Metric, F.Cu at (134.4, 105.3)
- added C112: 22pF, Capacitor_SMD:C_0402_1005Metric, F.Cu at (127.4, 101.0)
- added C113: 22pF, Capacitor_SMD:C_0402_1005Metric, F.Cu at (127.4, 102.9)
- added C114: 22u, Capacitor_SMD:C_1206_3216Metric, F.Cu at (128.8, 96.3)
- added C115: 10 nF, Capacitor_SMD:C_0603_1608Metric, F.Cu at (138.0, 117.4)
- added C116: 10 nF, Capacitor_SMD:C_0603_1608Metric, F.Cu at (138.0, 119.9)
- added C117: 10 nF, Capacitor_SMD:C_0603_1608Metric, F.Cu at (138.0, 122.4)
- added C118: 10 nF, Capacitor_SMD:C_0603_1608Metric, F.Cu at (138.0, 124.9)
- added C119: 10 nF, Capacitor_SMD:C_0603_1608Metric, F.Cu at (138.0, 127.4)
- added C12: 10 nF, Capacitor_SMD:C_0603_1608Metric, F.Cu at (109.9, 87.8)
- added C120: 10 nF, Capacitor_SMD:C_0603_1608Metric, F.Cu at (138.0, 129.9)
- added C121: 10 nF, Capacitor_SMD:C_0603_1608Metric, F.Cu at (116.5, 144.5)
- added C13: 10 nF, Capacitor_SMD:C_0603_1608Metric, F.Cu at (109.9, 90.3)
- added C14: 10 nF, Capacitor_SMD:C_0603_1608Metric, F.Cu at (109.9, 92.8)
- added C15: 10 nF, Capacitor_SMD:C_0603_1608Metric, F.Cu at (109.9, 95.3)
- added C16: 10 nF, Capacitor_SMD:C_0603_1608Metric, F.Cu at (109.9, 97.8)
- added C17: 10 nF, Capacitor_SMD:C_0603_1608Metric, F.Cu at (109.9, 100.3)
- added C18: 10 nF, Capacitor_SMD:C_0603_1608Metric, F.Cu at (109.9, 102.8)
- added C19: 10 nF, Capacitor_SMD:C_0603_1608Metric, F.Cu at (109.9, 105.3)
- added C2: 10 nF, Capacitor_SMD:C_0603_1608Metric, F.Cu at (105.9, 90.3)
- added C20: 10 nF, Capacitor_SMD:C_0603_1608Metric, F.Cu at (109.9, 107.8)
- added C21: 10 nF, Capacitor_SMD:C_0603_1608Metric, F.Cu at (109.9, 110.3)
- added C22: 10 nF, Capacitor_SMD:C_0603_1608Metric, F.Cu at (109.9, 112.8)
- added C23: 10 nF, Capacitor_SMD:C_0603_1608Metric, F.Cu at (77.8, 126.0)
- added C24: 10 nF, Capacitor_SMD:C_0603_1608Metric, F.Cu at (77.8, 128.5)
- added C25: 10 nF, Capacitor_SMD:C_0603_1608Metric, F.Cu at (77.8, 131.0)
- added C26: 10 nF, Capacitor_SMD:C_0603_1608Metric, F.Cu at (77.8, 133.5)
- added C27: 10 nF, Capacitor_SMD:C_0603_1608Metric, F.Cu at (77.8, 136.0)
- added C28: 10 nF, Capacitor_SMD:C_0603_1608Metric, F.Cu at (77.8, 138.5)
- added C29: 10 nF, Capacitor_SMD:C_0603_1608Metric, F.Cu at (77.8, 141.1)
- added C3: 10 nF, Capacitor_SMD:C_0603_1608Metric, F.Cu at (105.9, 92.8)
- added C30: 10 nF, Capacitor_SMD:C_0603_1608Metric, F.Cu at (77.8, 143.6)
- added C31: 10 nF, Capacitor_SMD:C_0603_1608Metric, F.Cu at (77.8, 146.1)
- added C32: 10 nF, Capacitor_SMD:C_0603_1608Metric, F.Cu at (77.8, 148.6)
- added C33: 10 nF, Capacitor_SMD:C_0603_1608Metric, F.Cu at (77.8, 151.1)
- added C34: 10 nF, Capacitor_SMD:C_0603_1608Metric, F.Cu at (81.8, 126.0)
- added C35: 10 nF, Capacitor_SMD:C_0603_1608Metric, F.Cu at (81.8, 128.5)
- added C36: 10 nF, Capacitor_SMD:C_0603_1608Metric, F.Cu at (81.8, 131.0)
- added C37: 10 nF, Capacitor_SMD:C_0603_1608Metric, F.Cu at (81.8, 133.5)
- added C38: 10 nF, Capacitor_SMD:C_0603_1608Metric, F.Cu at (81.8, 136.0)
- added C39: 10 nF, Capacitor_SMD:C_0603_1608Metric, F.Cu at (81.8, 138.5)
- added C4: 10 nF, Capacitor_SMD:C_0603_1608Metric, F.Cu at (105.9, 95.3)
- added C40: 10 nF, Capacitor_SMD:C_0603_1608Metric, F.Cu at (81.8, 141.1)
- added C41: 10 nF, Capacitor_SMD:C_0603_1608Metric, F.Cu at (81.8, 143.6)
- added C42: 10 nF, Capacitor_SMD:C_0603_1608Metric, F.Cu at (81.8, 146.1)
- added C43: 10 nF, Capacitor_SMD:C_0603_1608Metric, F.Cu at (81.8, 148.6)
- added C44: 10 nF, Capacitor_SMD:C_0603_1608Metric, F.Cu at (81.8, 151.1)
- added C45: 10 nF, Capacitor_SMD:C_0603_1608Metric, F.Cu at (132.0, 117.4)
- added C46: 10 nF, Capacitor_SMD:C_0603_1608Metric, F.Cu at (132.0, 119.9)
- added C47: 10 nF, Capacitor_SMD:C_0603_1608Metric, F.Cu at (132.0, 122.4)
- added C48: 10 nF, Capacitor_SMD:C_0603_1608Metric, F.Cu at (132.0, 124.9)
- added C49: 10 nF, Capacitor_SMD:C_0603_1608Metric, F.Cu at (105.9, 117.4)
- added C5: 10 nF, Capacitor_SMD:C_0603_1608Metric, F.Cu at (105.9, 97.8)
- added C50: 10 nF, Capacitor_SMD:C_0603_1608Metric, F.Cu at (105.9, 119.9)
- added C51: 10 nF, Capacitor_SMD:C_0603_1608Metric, F.Cu at (105.9, 122.4)
- added C52: 10 nF, Capacitor_SMD:C_0603_1608Metric, F.Cu at (105.9, 124.9)
- added C53: 10 nF, Capacitor_SMD:C_0603_1608Metric, F.Cu at (105.9, 127.4)
- added C54: 10 nF, Capacitor_SMD:C_0603_1608Metric, F.Cu at (105.9, 129.9)
- added C55: 10 nF, Capacitor_SMD:C_0603_1608Metric, F.Cu at (105.9, 132.4)
- added C56: 10 nF, Capacitor_SMD:C_0603_1608Metric, F.Cu at (105.9, 134.9)
- added C57: 10 nF, Capacitor_SMD:C_0603_1608Metric, F.Cu at (105.9, 137.4)
- added C58: 10 nF, Capacitor_SMD:C_0603_1608Metric, F.Cu at (105.9, 139.9)
- added C59: 10 nF, Capacitor_SMD:C_0603_1608Metric, F.Cu at (109.9, 117.4)
- added C6: 10 nF, Capacitor_SMD:C_0603_1608Metric, F.Cu at (105.9, 100.3)
- added C60: 10 nF, Capacitor_SMD:C_0603_1608Metric, F.Cu at (109.9, 119.9)
- added C61: 10 nF, Capacitor_SMD:C_0603_1608Metric, F.Cu at (109.9, 122.4)
- added C62: 10 nF, Capacitor_SMD:C_0603_1608Metric, F.Cu at (109.9, 124.9)
- added C63: 10 nF, Capacitor_SMD:C_0603_1608Metric, F.Cu at (109.9, 127.4)
- added C64: 10 nF, Capacitor_SMD:C_0603_1608Metric, F.Cu at (109.9, 129.9)
- added C65: 10 nF, Capacitor_SMD:C_0603_1608Metric, F.Cu at (109.9, 132.4)
- added C66: 10 nF, Capacitor_SMD:C_0603_1608Metric, F.Cu at (109.9, 134.9)
- added C67: 10 nF, Capacitor_SMD:C_0603_1608Metric, F.Cu at (109.9, 137.4)
- added C68: 10 nF, Capacitor_SMD:C_0603_1608Metric, F.Cu at (109.9, 139.9)
- added C69: 10 nF, Capacitor_SMD:C_0603_1608Metric, F.Cu at (113.9, 117.4)
- added C7: 10 nF, Capacitor_SMD:C_0603_1608Metric, F.Cu at (105.9, 102.8)
- added C70: 10 nF, Capacitor_SMD:C_0603_1608Metric, F.Cu at (113.9, 119.9)
- added C71: 10 nF, Capacitor_SMD:C_0603_1608Metric, F.Cu at (113.9, 122.4)
- added C72: 10 nF, Capacitor_SMD:C_0603_1608Metric, F.Cu at (113.9, 124.9)
- added C73: 10 nF, Capacitor_SMD:C_0603_1608Metric, F.Cu at (113.9, 127.4)
- added C74: 10 nF, Capacitor_SMD:C_0603_1608Metric, F.Cu at (113.9, 129.9)
- added C75: 10 nF, Capacitor_SMD:C_0603_1608Metric, F.Cu at (113.9, 132.4)
- added C76: 10 nF, Capacitor_SMD:C_0603_1608Metric, F.Cu at (113.9, 134.9)
- added C77: 10 nF, Capacitor_SMD:C_0603_1608Metric, F.Cu at (113.9, 137.4)
- added C78: 10 nF, Capacitor_SMD:C_0603_1608Metric, F.Cu at (113.9, 139.9)
- added C79: 10 nF, Capacitor_SMD:C_0603_1608Metric, F.Cu at (118.0, 117.4)
- added C8: 10 nF, Capacitor_SMD:C_0603_1608Metric, F.Cu at (105.9, 105.3)
- added C80: 10 nF, Capacitor_SMD:C_0603_1608Metric, F.Cu at (118.0, 119.9)
- added C81: 10 nF, Capacitor_SMD:C_0603_1608Metric, F.Cu at (77.8, 87.8)
- added C82: 22pF, Capacitor_SMD:C_0402_1005Metric, F.Cu at (99.0, 110.1)
- added C83: 10 nF, Capacitor_SMD:C_0603_1608Metric, F.Cu at (77.8, 90.3)
- added C84: 10 nF, Capacitor_SMD:C_0603_1608Metric, F.Cu at (77.8, 92.8)
- added C85: 10 nF, Capacitor_SMD:C_0603_1608Metric, F.Cu at (77.8, 95.3)
- added C86: 10 nF, Capacitor_SMD:C_0603_1608Metric, F.Cu at (77.8, 97.8)
- added C87: 10 nF, Capacitor_SMD:C_0603_1608Metric, F.Cu at (77.8, 100.3)
- added C88: 22pF, Capacitor_SMD:C_0402_1005Metric, F.Cu at (99.0, 112.0)
- added C89: 10 nF, Capacitor_SMD:C_0603_1608Metric, F.Cu at (77.8, 102.8)
- added C9: 10 nF, Capacitor_SMD:C_0603_1608Metric, F.Cu at (105.9, 107.8)
- added C90: 10 nF, Capacitor_SMD:C_0603_1608Metric, F.Cu at (77.8, 105.3)
- added C91: 10 nF, Capacitor_SMD:C_0603_1608Metric, F.Cu at (77.8, 107.8)
- added C92: 10 nF, Capacitor_SMD:C_0603_1608Metric, F.Cu at (81.8, 87.8)
- added C93: 10 nF, Capacitor_SMD:C_0603_1608Metric, F.Cu at (81.8, 90.3)
- added C94: 10 nF, Capacitor_SMD:C_0603_1608Metric, F.Cu at (81.8, 92.8)
- added C95: 10 nF, Capacitor_SMD:C_0603_1608Metric, F.Cu at (81.8, 95.3)
- added C96: 22pF, Capacitor_SMD:C_0402_1005Metric, F.Cu at (99.0, 114.0)
- added C97: 10 nF, Capacitor_SMD:C_0603_1608Metric, F.Cu at (81.8, 97.8)
- added C98: 10 nF, Capacitor_SMD:C_0603_1608Metric, F.Cu at (81.8, 100.3)
- added C99: 22pF, Capacitor_SMD:C_0402_1005Metric, F.Cu at (99.0, 116.0)
- added D10: Schottky_100V_1A, Diode_SMD:D_PowerDI-123, F.Cu at (98.9, 99.3)
- added D2: Schottky_100V_1A, Diode_SMD:D_PowerDI-123, F.Cu at (98.9, 88.3)
- added D3: Schottky_100V_1A, Diode_SMD:D_PowerDI-123, F.Cu at (98.9, 92.0)
- added D4: PTVS60VS1UR, Diode_SMD:Nexperia_CFP3_SOD-123W, F.Cu at (98.7, 102.7)
- added D5: S1MSP1-7, Diode_SMD:D_PowerDI-123, F.Cu at (98.9, 95.6)
- added D6: PESD5V0V1BB, Diode_SMD:D_SOD-523, F.Cu at (95.8, 110.3)
- added D7: PESD5V0V1BB, Diode_SMD:D_SOD-523, F.Cu at (95.8, 112.8)
- added D8: PESD5V0V1BB, Diode_SMD:D_SOD-523, F.Cu at (95.8, 115.2)
- added D9: PESD5V0V1BB, Diode_SMD:D_SOD-523, F.Cu at (95.8, 117.7)
- added GND1: Testpoint_Square, TestPoint:TestPoint_Pad_2.5x2.5mm, F.Cu at (78.1, 120.5)
- added IC1: MCP9800A0T-M/OT, Package_TO_SOT_SMD:SOT-23-5, F.Cu at (142.6, 118.5)
- added J10: Pinheader_2x7_vertical, Connector_PinHeader_2.54mm:PinHeader_2x07_P2.54mm_Vertical, F.Cu at (144.6, 150.6)
- added J11: Pinheader_2x1_vertical, Connector_PinHeader_2.54mm:PinHeader_1x02_P2.54mm_Vertical, F.Cu at (136.9, 140.5)
- added J12: Pinheader_2x1_vertical, Connector_PinHeader_2.54mm:PinHeader_1x02_P2.54mm_Vertical, F.Cu at (141.4, 140.5)
- added J13: Pinheader_2x9_vertical, Connector_PinHeader_2.54mm:PinHeader_2x09_P2.54mm_Vertical, F.Cu at (128.0, 150.5)
- added J2: Pinheader_2x1_vertical, Connector_PinHeader_2.54mm:PinHeader_1x02_P2.54mm_Vertical, F.Cu at (132.3, 140.5)
- added J9: Pinheader_2x7_vertical, Connector_PinHeader_2.54mm:PinHeader_2x07_P2.54mm_Vertical, F.Cu at (136.0, 151.1)
- added L1: 470nH, Inductor_SMD:L_Bourns_SRP7028A_7.3x6.6mm, F.Cu at (130.9, 90.6)
- added R1: 0, Resistor_SMD:R_0603_1608Metric, F.Cu at (116.5, 151.5)
- added R10: 0, Resistor_SMD:R_0603_1608Metric, F.Cu at (113.9, 107.8)
- added R11: 0, Resistor_SMD:R_0603_1608Metric, F.Cu at (113.9, 110.3)
- added R110: 0, Resistor_SMD:R_0603_1608Metric, F.Cu at (118.0, 122.4)
- added R111: 0, Resistor_SMD:R_0603_1608Metric, F.Cu at (118.0, 124.9)
- added R112: 0, Resistor_SMD:R_0603_1608Metric, F.Cu at (118.0, 127.4)
- added R113: 0, Resistor_SMD:R_0603_1608Metric, F.Cu at (118.0, 129.9)
- added R114: 0, Resistor_SMD:R_0603_1608Metric, F.Cu at (118.0, 132.4)
- added R115: 0, Resistor_SMD:R_0603_1608Metric, F.Cu at (118.0, 134.9)
- added R116: 0, Resistor_SMD:R_0603_1608Metric, F.Cu at (118.0, 137.4)
- added R117: 0, Resistor_SMD:R_0603_1608Metric, F.Cu at (118.0, 139.9)
- added R118: 10K, Resistor_SMD:R_0603_1608Metric, F.Cu at (122.0, 117.4)
- added R119: 10K, Resistor_SMD:R_0603_1608Metric, F.Cu at (122.0, 119.9)
- added R12: 1K, Resistor_SMD:R_0603_1608Metric, F.Cu at (113.9, 112.8)
- added R120: 10K, Resistor_SMD:R_0603_1608Metric, F.Cu at (122.0, 122.4)
- added R121: 10K, Resistor_SMD:R_0603_1608Metric, F.Cu at (122.0, 124.9)
- added R122: 10K, Resistor_SMD:R_0603_1608Metric, F.Cu at (122.0, 127.4)
- added R123: 10K, Resistor_SMD:R_0603_1608Metric, F.Cu at (122.0, 129.9)
- added R124: 10K, Resistor_SMD:R_0603_1608Metric, F.Cu at (122.0, 132.4)
- added R125: 10K, Resistor_SMD:R_0603_1608Metric, F.Cu at (122.0, 134.9)
- added R126: 0, Resistor_SMD:R_0603_1608Metric, F.Cu at (122.0, 137.4)
- added R127: 0, Resistor_SMD:R_0603_1608Metric, F.Cu at (122.0, 139.9)
- added R128: 0, Resistor_SMD:R_0603_1608Metric, F.Cu at (126.0, 117.4)
- added R129: 10K, Resistor_SMD:R_0603_1608Metric, F.Cu at (126.0, 119.9)
- added R13: 1K, Resistor_SMD:R_0603_1608Metric, F.Cu at (118.0, 87.8)
- added R130: 10K, Resistor_SMD:R_0603_1608Metric, F.Cu at (126.0, 122.4)
- added R131: 10K, Resistor_SMD:R_0603_1608Metric, F.Cu at (126.0, 124.9)
- added R132: 10K, Resistor_SMD:R_0603_1608Metric, F.Cu at (126.0, 127.4)
- added R133: 10K, Resistor_SMD:R_0603_1608Metric, F.Cu at (126.0, 129.9)
- added R134: 10K, Resistor_SMD:R_0603_1608Metric, F.Cu at (126.0, 132.4)
- added R135: 10K, Resistor_SMD:R_0603_1608Metric, F.Cu at (126.0, 134.9)
- added R136: 10K, Resistor_SMD:R_0603_1608Metric, F.Cu at (126.0, 137.4)
- added R139: 0, Resistor_SMD:R_0603_1608Metric, F.Cu at (81.8, 102.8)
- added R14: 1K, Resistor_SMD:R_0603_1608Metric, F.Cu at (118.0, 90.3)
- added R140: 0, Resistor_SMD:R_0603_1608Metric, F.Cu at (81.8, 105.3)
- added R141: 0, Resistor_SMD:R_0603_1608Metric, F.Cu at (81.8, 107.8)
- added R142: 0, Resistor_SMD:R_0603_1608Metric, F.Cu at (85.8, 87.8)
- added R143: 0, Resistor_SMD:R_0603_1608Metric, F.Cu at (85.8, 90.3)
- added R144: 0, Resistor_SMD:R_0603_1608Metric, F.Cu at (85.8, 92.8)
- added R145: 0, Resistor_SMD:R_0603_1608Metric, F.Cu at (85.8, 95.3)
- added R146: 0, Resistor_SMD:R_0603_1608Metric, F.Cu at (85.8, 97.8)
- added R147: 0, Resistor_SMD:R_0603_1608Metric, F.Cu at (85.8, 100.3)
- added R148: 0, Resistor_SMD:R_0603_1608Metric, F.Cu at (85.8, 102.8)
- added R149: 0, Resistor_SMD:R_0603_1608Metric, F.Cu at (85.8, 105.3)
- added R15: 1K, Resistor_SMD:R_0603_1608Metric, F.Cu at (118.0, 92.8)
- added R150: 0, Resistor_SMD:R_0603_1608Metric, F.Cu at (85.8, 107.8)
- added R151: 0, Resistor_SMD:R_0603_1608Metric, F.Cu at (89.8, 87.8)
- added R152: 0, Resistor_SMD:R_0603_1608Metric, F.Cu at (89.8, 90.3)
- added R153: 0, Resistor_SMD:R_0603_1608Metric, F.Cu at (89.8, 92.8)
- added R154: 0, Resistor_SMD:R_0603_1608Metric, F.Cu at (89.8, 95.3)
- added R155: 0, Resistor_SMD:R_0603_1608Metric, F.Cu at (89.8, 97.8)
- added R156: 0, Resistor_SMD:R_0603_1608Metric, F.Cu at (89.8, 100.3)
- added R157: 0, Resistor_SMD:R_0603_1608Metric, F.Cu at (89.8, 102.8)
- added R158: 0, Resistor_SMD:R_0603_1608Metric, F.Cu at (89.8, 105.3)
- added R16: 1K, Resistor_SMD:R_0603_1608Metric, F.Cu at (118.0, 95.3)
- added R162: 0, Resistor_SMD:R_0603_1608Metric, F.Cu at (89.8, 107.8)
- added R17: 1K, Resistor_SMD:R_0603_1608Metric, F.Cu at (118.0, 97.8)
- added R170: 0, Resistor_SMD:R_0603_1608Metric, F.Cu at (93.9, 87.8)
- added R174: 0, Resistor_SMD:R_0603_1608Metric, F.Cu at (93.9, 90.3)
- added R176: 0, Resistor_SMD:R_0603_1608Metric, F.Cu at (93.9, 92.8)
- added R177: 0, Resistor_SMD:R_0603_1608Metric, F.Cu at (93.9, 95.3)
- added R178: 0, Resistor_SMD:R_0603_1608Metric, F.Cu at (93.9, 97.8)
- added R179: 0, Resistor_SMD:R_0603_1608Metric, F.Cu at (93.9, 100.3)
- added R18: 1K, Resistor_SMD:R_0603_1608Metric, F.Cu at (118.0, 100.3)
- added R180: 0, Resistor_SMD:R_0603_1608Metric, F.Cu at (93.9, 102.8)
- added R181: 0, Resistor_SMD:R_0603_1608Metric, F.Cu at (105.9, 149.5)
- added R183: 0, Resistor_SMD:R_0603_1608Metric, F.Cu at (105.9, 152.0)
- added R185: 0, Resistor_SMD:R_0603_1608Metric, F.Cu at (105.9, 154.5)
- added R189: 0, Resistor_SMD:R_0603_1608Metric, F.Cu at (143.8, 98.4)
- added R19: 1K, Resistor_SMD:R_0603_1608Metric, F.Cu at (118.0, 102.8)
- added R190: 10K, Resistor_SMD:R_0603_1608Metric, F.Cu at (143.8, 100.9)
- added R191: 0, Resistor_SMD:R_0603_1608Metric, F.Cu at (143.8, 103.4)
- added R195: 0, Resistor_SMD:R_0603_1608Metric, F.Cu at (143.8, 105.9)
- added R199: 10K, Resistor_SMD:R_0603_1608Metric, F.Cu at (138.0, 132.4)
- added R2: 10K, Resistor_SMD:R_0603_1608Metric, F.Cu at (113.9, 87.8)
- added R20: 0, Resistor_SMD:R_0603_1608Metric, F.Cu at (118.0, 105.3)
- added R200: 10K, Resistor_SMD:R_0603_1608Metric, F.Cu at (116.5, 147.0)
- added R21: 0, Resistor_SMD:R_0603_1608Metric, F.Cu at (118.0, 107.8)
- added R22: 0, Resistor_SMD:R_0603_1608Metric, F.Cu at (118.0, 110.3)
- added R23: 0, Resistor_SMD:R_0603_1608Metric, F.Cu at (118.0, 112.8)
- added R24: 0, Resistor_SMD:R_0603_1608Metric, F.Cu at (122.0, 87.8)
- added R25: 0, Resistor_SMD:R_0603_1608Metric, F.Cu at (122.0, 90.3)
- added R26: 0, Resistor_SMD:R_0603_1608Metric, F.Cu at (122.0, 92.8)
- added R27: 0, Resistor_SMD:R_0603_1608Metric, F.Cu at (122.0, 95.3)
- added R28: 0, Resistor_SMD:R_0603_1608Metric, F.Cu at (122.0, 97.8)
- added R29: 0, Resistor_SMD:R_0603_1608Metric, F.Cu at (122.0, 100.3)
- added R3: 10K, Resistor_SMD:R_0603_1608Metric, F.Cu at (113.9, 90.3)
- added R30: 0, Resistor_SMD:R_0603_1608Metric, F.Cu at (122.0, 102.8)
- added R31: 1K, Resistor_SMD:R_0603_1608Metric, F.Cu at (122.0, 105.3)
- added R32: 0, Resistor_SMD:R_0603_1608Metric, F.Cu at (122.0, 107.8)
- added R33: 0, Resistor_SMD:R_0603_1608Metric, F.Cu at (122.0, 110.3)
- added R34: 0, Resistor_SMD:R_0603_1608Metric, F.Cu at (122.0, 112.8)
- added R35: 10K, Resistor_SMD:R_0603_1608Metric, F.Cu at (85.8, 126.0)
- added R36: 10K, Resistor_SMD:R_0603_1608Metric, F.Cu at (85.8, 128.5)
- added R37: 10K, Resistor_SMD:R_0603_1608Metric, F.Cu at (85.8, 131.0)
- added R38: 10K, Resistor_SMD:R_0603_1608Metric, F.Cu at (85.8, 133.5)
- added R39: 10K, Resistor_SMD:R_0603_1608Metric, F.Cu at (85.8, 136.0)
- added R4: 10K, Resistor_SMD:R_0603_1608Metric, F.Cu at (113.9, 92.8)
- added R40: 10K, Resistor_SMD:R_0603_1608Metric, F.Cu at (85.8, 138.5)
- added R41: 10K, Resistor_SMD:R_0603_1608Metric, F.Cu at (85.8, 141.1)
- added R42: 10K, Resistor_SMD:R_0603_1608Metric, F.Cu at (85.8, 143.6)
- added R43: 0, Resistor_SMD:R_0603_1608Metric, F.Cu at (85.8, 146.1)
- added R44: 0, Resistor_SMD:R_0603_1608Metric, F.Cu at (85.8, 148.6)
- added R45: 1K, Resistor_SMD:R_0603_1608Metric, F.Cu at (85.8, 151.1)
- added R46: 1K, Resistor_SMD:R_0603_1608Metric, F.Cu at (89.8, 126.0)
- added R47: 1K, Resistor_SMD:R_0603_1608Metric, F.Cu at (89.8, 128.5)
- added R48: 1K, Resistor_SMD:R_0603_1608Metric, F.Cu at (89.8, 131.0)
- added R49: 1K, Resistor_SMD:R_0603_1608Metric, F.Cu at (89.8, 133.5)
- added R5: 10K, Resistor_SMD:R_0603_1608Metric, F.Cu at (113.9, 95.3)
- added R50: 1K, Resistor_SMD:R_0603_1608Metric, F.Cu at (89.8, 136.0)
- added R51: 1K, Resistor_SMD:R_0603_1608Metric, F.Cu at (89.8, 138.5)
- added R52: 1K, Resistor_SMD:R_0603_1608Metric, F.Cu at (89.8, 141.1)
- added R53: 0, Resistor_SMD:R_0603_1608Metric, F.Cu at (89.8, 143.6)
- added R54: 0, Resistor_SMD:R_0603_1608Metric, F.Cu at (89.8, 146.1)
- added R55: 0, Resistor_SMD:R_0603_1608Metric, F.Cu at (89.8, 148.6)
- added R56: 0, Resistor_SMD:R_0603_1608Metric, F.Cu at (89.8, 151.1)
- added R57: 0, Resistor_SMD:R_0603_1608Metric, F.Cu at (93.9, 126.0)
- added R58: 0, Resistor_SMD:R_0603_1608Metric, F.Cu at (93.9, 128.5)
- added R59: 0, Resistor_SMD:R_0603_1608Metric, F.Cu at (93.9, 131.0)
- added R6: 10K, Resistor_SMD:R_0603_1608Metric, F.Cu at (113.9, 97.8)
- added R60: 0, Resistor_SMD:R_0603_1608Metric, F.Cu at (93.9, 133.5)
- added R61: 0, Resistor_SMD:R_0603_1608Metric, F.Cu at (93.9, 136.0)
- added R62: 0, Resistor_SMD:R_0603_1608Metric, F.Cu at (93.9, 138.5)
- added R63: 0, Resistor_SMD:R_0603_1608Metric, F.Cu at (93.9, 141.1)
- added R64: 1K, Resistor_SMD:R_0603_1608Metric, F.Cu at (93.9, 143.6)
- added R65: 0, Resistor_SMD:R_0603_1608Metric, F.Cu at (93.9, 146.1)
- added R66: 0, Resistor_SMD:R_0603_1608Metric, F.Cu at (93.9, 148.6)
- added R67: 0, Resistor_SMD:R_0603_1608Metric, F.Cu at (93.9, 151.1)
- added R7: 10K, Resistor_SMD:R_0603_1608Metric, F.Cu at (113.9, 100.3)
- added R79: 10K, Resistor_SMD:R_0603_1608Metric, F.Cu at (132.0, 127.4)
- added R8: 10K, Resistor_SMD:R_0603_1608Metric, F.Cu at (113.9, 102.8)
- added R83: 10K, Resistor_SMD:R_0603_1608Metric, F.Cu at (132.0, 129.9)
- added R89: 10K, Resistor_SMD:R_0603_1608Metric, F.Cu at (132.0, 132.4)
- added R9: 10K, Resistor_SMD:R_0603_1608Metric, F.Cu at (113.9, 105.3)
- added R93: 10K, Resistor_SMD:R_0603_1608Metric, F.Cu at (132.0, 134.9)
- added TPL_H_N1: Testpoint_Square, TestPoint:TestPoint_Pad_2.5x2.5mm, F.Cu at (82.6, 111.4)
- added TPL_H_P1: Testpoint_Square, TestPoint:TestPoint_Pad_2.5x2.5mm, F.Cu at (82.6, 115.9)
- added TPL_L_N1: Testpoint_Square, TestPoint:TestPoint_Pad_2.5x2.5mm, F.Cu at (82.6, 120.5)
- added TPL_L_P1: Testpoint_Square, TestPoint:TestPoint_Pad_2.5x2.5mm, F.Cu at (87.2, 111.4)
- added Vaux1: Testpoint_Square, TestPoint:TestPoint_Pad_2.5x2.5mm, F.Cu at (87.2, 115.9)
- added Vbat1: Testpoint_Square, TestPoint:TestPoint_Pad_2.5x2.5mm, F.Cu at (87.2, 120.5)
- added Vbat_con_ext1: Testpoint_Square, TestPoint:TestPoint_Pad_2.5x2.5mm, F.Cu at (91.7, 111.4)
- added Vddc1: Testpoint_Square, TestPoint:TestPoint_Pad_2.5x2.5mm, F.Cu at (91.7, 115.9)
- added Vin_DCDC1: Testpoint_Square, TestPoint:TestPoint_Pad_2.5x2.5mm, F.Cu at (139.5, 101.5)
- added Vmodule1: Testpoint_Square, TestPoint:TestPoint_Pad_2.5x2.5mm, F.Cu at (91.7, 120.5)
- added enable_DCDC1: Testpoint_Square, TestPoint:TestPoint_Pad_2.5x2.5mm, F.Cu at (139.5, 106.0)
Routing:
- net (no net): track 0.00 -> 92.3 mm, vias 0 -> 1066
- net BAL.CB_HI14: track 10.4 -> 0.00 mm, vias 34 -> 0
- net BAL.CB_LO12: track 10.1 -> 0.00 mm, vias 34 -> 0
- net CIN14: track 10.0 -> 0.00 mm, vias 52 -> 0
- net CIN12: track 8.49 -> 0.00 mm, vias 81 -> 0
- net BAL.CB_HI8: track 7.63 -> 0.00 mm, vias 34 -> 0
- net BAL.CB_LO2: track 7.01 -> 0.00 mm, vias 34 -> 0
- net BAL.CB_HI12: track 6.44 -> 0.00 mm, vias 34 -> 0
- net BAL.CB_LO6: track 5.84 -> 0.00 mm, vias 34 -> 0
- net BAL.CB_HI10: track 4.94 -> 0.00 mm, vias 34 -> 0
- net CIN10: track 4.91 -> 0.00 mm, vias 81 -> 0
- net BAL.CB_LO4: track 4.45 -> 0.00 mm, vias 34 -> 0
- net BAL.CB_LO8: track 2.88 -> 0.00 mm, vias 34 -> 0
- net BAL.CB_LO10: track 2.75 -> 0.00 mm, vias 34 -> 0
- net CIN0: track 2.51 -> 0.00 mm, vias 52 -> 0
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- added copper zone on B.Cu, net (none)
- added copper zone on F.Cu, net (none)
- added copper zone on In1.Cu, net (none)
- added copper zone on In2.Cu, net (none)
- added copper zone on In3.Cu, net (none)
- added copper zone on In4.Cu, net (none)
- removed copper zone on B.Cu, net BAL.CB_HI10
- removed copper zone on F.Cu, net BAL.CB_HI10
- removed copper zone on In1.Cu, net BAL.CB_HI10
- removed copper zone on In2.Cu, net BAL.CB_HI10
- removed copper zone on In3.Cu, net BAL.CB_HI10
- removed copper zone on In4.Cu, net BAL.CB_HI10
- removed copper zone on B.Cu, net BAL.CB_HI12
- removed copper zone on F.Cu, net BAL.CB_HI12
- removed copper zone on In1.Cu, net BAL.CB_HI12
- removed copper zone on In2.Cu, net BAL.CB_HI12
- removed copper zone on In3.Cu, net BAL.CB_HI12
- removed copper zone on In4.Cu, net BAL.CB_HI12
- removed copper zone on B.Cu, net BAL.CB_HI14
- removed copper zone on F.Cu, net BAL.CB_HI14
- removed copper zone on In1.Cu, net BAL.CB_HI14
- removed copper zone on In2.Cu, net BAL.CB_HI14
- removed copper zone on In3.Cu, net BAL.CB_HI14
- removed copper zone on In4.Cu, net BAL.CB_HI14
- removed copper zone on B.Cu, net BAL.CB_HI2
- removed copper zone on F.Cu, net BAL.CB_HI2
- removed copper zone on In1.Cu, net BAL.CB_HI2
- removed copper zone on In2.Cu, net BAL.CB_HI2
- removed copper zone on In3.Cu, net BAL.CB_HI2
- removed copper zone on In4.Cu, net BAL.CB_HI2
- removed copper zone on B.Cu, net BAL.CB_HI4
- removed copper zone on F.Cu, net BAL.CB_HI4
- removed copper zone on In1.Cu, net BAL.CB_HI4
- removed copper zone on In2.Cu, net BAL.CB_HI4
- removed copper zone on In3.Cu, net BAL.CB_HI4
- removed copper zone on In4.Cu, net BAL.CB_HI4
- removed copper zone on B.Cu, net BAL.CB_HI6
- removed copper zone on F.Cu, net BAL.CB_HI6
- removed copper zone on In1.Cu, net BAL.CB_HI6
- removed copper zone on In2.Cu, net BAL.CB_HI6
- removed copper zone on In3.Cu, net BAL.CB_HI6
- removed copper zone on In4.Cu, net BAL.CB_HI6
- removed copper zone on B.Cu, net BAL.CB_HI8
- removed copper zone on F.Cu, net BAL.CB_HI8
- removed copper zone on In1.Cu, net BAL.CB_HI8
- removed copper zone on In2.Cu, net BAL.CB_HI8
- removed copper zone on In3.Cu, net BAL.CB_HI8
- removed copper zone on In4.Cu, net BAL.CB_HI8
- removed copper zone on B.Cu, net BAL.CB_LO0
- removed copper zone on F.Cu, net BAL.CB_LO0
- removed copper zone on In1.Cu, net BAL.CB_LO0
- removed copper zone on In2.Cu, net BAL.CB_LO0
- removed copper zone on In3.Cu, net BAL.CB_LO0
- removed copper zone on In4.Cu, net BAL.CB_LO0
- removed copper zone on B.Cu, net BAL.CB_LO10
- removed copper zone on F.Cu, net BAL.CB_LO10
- removed copper zone on In1.Cu, net BAL.CB_LO10
- removed copper zone on In2.Cu, net BAL.CB_LO10
- removed copper zone on In3.Cu, net BAL.CB_LO10
- removed copper zone on In4.Cu, net BAL.CB_LO10
- removed copper zone on B.Cu, net BAL.CB_LO12
- removed copper zone on F.Cu, net BAL.CB_LO12
- removed copper zone on In1.Cu, net BAL.CB_LO12
- removed copper zone on In2.Cu, net BAL.CB_LO12
- removed copper zone on In3.Cu, net BAL.CB_LO12
- removed copper zone on In4.Cu, net BAL.CB_LO12
- removed copper zone on B.Cu, net BAL.CB_LO2
- removed copper zone on F.Cu, net BAL.CB_LO2
- removed copper zone on In1.Cu, net BAL.CB_LO2
- removed copper zone on In2.Cu, net BAL.CB_LO2
- removed copper zone on In3.Cu, net BAL.CB_LO2
- removed copper zone on In4.Cu, net BAL.CB_LO2
- removed copper zone on B.Cu, net BAL.CB_LO4
- removed copper zone on F.Cu, net BAL.CB_LO4
- removed copper zone on In1.Cu, net BAL.CB_LO4
- removed copper zone on In2.Cu, net BAL.CB_LO4
- removed copper zone on In3.Cu, net BAL.CB_LO4
- removed copper zone on In4.Cu, net BAL.CB_LO4
- removed copper zone on B.Cu, net BAL.CB_LO6
- removed copper zone on F.Cu, net BAL.CB_LO6
- removed copper zone on In1.Cu, net BAL.CB_LO6
- removed copper zone on In2.Cu, net BAL.CB_LO6
- removed copper zone on In3.Cu, net BAL.CB_LO6
- removed copper zone on In4.Cu, net BAL.CB_LO6
- removed copper zone on B.Cu, net BAL.CB_LO8
- removed copper zone on F.Cu, net BAL.CB_LO8
- removed copper zone on In1.Cu, net BAL.CB_LO8
- removed copper zone on In2.Cu, net BAL.CB_LO8
- removed copper zone on In3.Cu, net BAL.CB_LO8
- removed copper zone on In4.Cu, net BAL.CB_LO8
- removed copper zone on B.Cu, net CIN0
- removed copper zone on F.Cu, net CIN0
- removed copper zone on In1.Cu, net CIN0
- removed copper zone on In2.Cu, net CIN0
- removed copper zone on In3.Cu, net CIN0
- removed copper zone on In4.Cu, net CIN0
- removed copper zone on B.Cu, net CIN10
- removed copper zone on F.Cu, net CIN10
- removed copper zone on In1.Cu, net CIN10
- removed copper zone on In2.Cu, net CIN10
- removed copper zone on In3.Cu, net CIN10
- removed copper zone on In4.Cu, net CIN10
- removed copper zone on B.Cu, net CIN12
- removed copper zone on F.Cu, net CIN12
- removed copper zone on In1.Cu, net CIN12
- removed copper zone on In2.Cu, net CIN12
- removed copper zone on In3.Cu, net CIN12
- removed copper zone on In4.Cu, net CIN12
- removed copper zone on B.Cu, net CIN14
- removed copper zone on F.Cu, net CIN14
- removed copper zone on In1.Cu, net CIN14
- removed copper zone on In2.Cu, net CIN14
- removed copper zone on In3.Cu, net CIN14
- removed copper zone on In4.Cu, net CIN14
- removed copper zone on B.Cu, net CIN2
- removed copper zone on F.Cu, net CIN2
- removed copper zone on In1.Cu, net CIN2
- removed copper zone on In2.Cu, net CIN2
- removed copper zone on In3.Cu, net CIN2
- removed copper zone on In4.Cu, net CIN2
- removed copper zone on B.Cu, net CIN4
- removed copper zone on F.Cu, net CIN4
- removed copper zone on In1.Cu, net CIN4
- removed copper zone on In2.Cu, net CIN4
- removed copper zone on In3.Cu, net CIN4
- removed copper zone on In4.Cu, net CIN4
- removed copper zone on B.Cu, net CIN6
- removed copper zone on F.Cu, net CIN6
- removed copper zone on In1.Cu, net CIN6
- removed copper zone on In2.Cu, net CIN6
- removed copper zone on In3.Cu, net CIN6
- removed copper zone on In4.Cu, net CIN6
- removed copper zone on B.Cu, net CIN8
- removed copper zone on F.Cu, net CIN8
- removed copper zone on In1.Cu, net CIN8
- removed copper zone on In2.Cu, net CIN8
- removed copper zone on In3.Cu, net CIN8
- removed copper zone on In4.Cu, net CIN8
